File: relayboard.sch (KiCad schematic (older format))
At the start: 23 parts, among them IC1 AT24C256C-SSHL-T, K1 RELAY_1RT, P1 Supply, P2 HLK-PM01, P3 Sensors Unleashed Radio, P4 Relay, Q1 FDN304P, Q2 BC849, U1 AMS1117

Commit message: Recalculated the mains detect circuit
Parts:
- R1, R2, R3: value 330k -> 549k
- R11: value 12835R -> 18.7k
- R4: value 6040R -> 4.99k
Changed lines of the file:
@@
 P 1700 2050
 F 0 "R1" V 1780 2050 50  0000 C CNN
-F 1 "330k" V 1700 2050 50  0000 C CNN
+F 1 "549k" V 1700 2050 50  0000 C CNN
 F 2 "Resistors_SMD:R_0805" V 1630 2050 50  0001 C CNN
-F 3 "https://industrial.panasonic.com/ww/products/resistors/chip-resistors/chip-resistors/anti-sulfurated-thick-film-chip-resistors/ERJS1DF3303U" H 1700 2050 50  0001 C CNN
+F 3 "" H 1700 2050 50  0001 C CNN
 F 4 "1%," H 1700 2050 60  0001 C CNN "Characteristics"
 F 5 "0805" H 1700 2050 60  0001 C CNN "Package ID"
@@
 P 3000 2350
 F 0 "R4" V 2900 2350 50  0000 C CNN
-F 1 "6040R" V 3100 2350 50  0000 C CNN
+F 1 "4.99k" V 3100 2350 50  0000 C CNN
 F 2 "Resistors_SMD:R_0805" V 2930 2350 50  0001 C CNN
 F 3 "" H 3000 2350 50  0001 C CNN
@@
 P 2050 2050
 F 0 "R2" V 2130 2050 50  0000 C CNN
-F 1 "330k" V 2050 2050 50  0000 C CNN
+F 1 "549k" V 2050 2050 50  0000 C CNN
 F 2 "Resistors_SMD:R_0805" V 1980 2050 50  0001 C CNN
 F 3 "https://industrial.panasonic.com/ww/products/resistors/chip-resistors/chip-resistors/anti-sulfurated-thick-film-chip-resistors/ERJS1DF3303U" H 2050 2050 50  0001 C CNN
@@
 P 2450 2050
 F 0 "R3" V 2530 2050 50  0000 C CNN
-F 1 "330k" V 2450 2050 50  0000 C CNN
+F 1 "549k" V 2450 2050 50  0000 C CNN
 F 2 "Resistors_SMD:R_0805" V 2380 2050 50  0001 C CNN
 F 3 "https://industrial.panasonic.com/ww/products/resistors/chip-resistors/chip-resistors/anti-sulfurated-thick-film-chip-resistors/ERJS1DF3303U" H 2450 2050 50  0001 C CNN
@@
 P 3000 1800
 F 0 "R11" V 2900 1800 50  0000 C CNN
-F 1 "12835R" V 3100 1800 50  0000 C CNN
+F 1 "18.7k" V 3100 1800 50  0000 C CNN
 F 2 "Resistors_SMD:R_0805" V 2930 1800 50  0001 C CNN
 F 3 "" H 3000 1800 50  0001 C CNN
